File: pcb/aup/ethernet.kicad_sch (KiCad schematic)
At the start: 2 parts, among them IC2 88E1512-A0-NNP2C000

Commit message: Update footprints and 3d models. All render
Parts:
- IC2: footprint !Misc:QFN50P800X800X100-57N-D -> !Misc:88E1512-A0-NNP2C000
Changed lines of the file:
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@@
 			)
 		)
-		(property "Footprint" "!Misc:QFN50P800X800X100-57N-D"
+		(property "Footprint" "!Misc:88E1512-A0-NNP2C000"
 			(at 83.82 133.02 0)
 			(effects
