File: pcb/aup/power_reg.kicad_sch (KiCad schematic)
At the start: 54 parts, among them U4 TPS563257DRLR, U5 TPS563257DRLR, U7 TPS563257DRLR, U8 TPS563257DRLR, U9 TPS563257DRLR

Commit message: First pass on lower rails
Connections:
- net FB_Vccint: now also R30.2, R31.1, U8.6 (FB)
- net FB_1V35: now reaches R26.2, R27.1, U7.6 (FB)
- net FB_3V3: now reaches R33.2, R34.1, U9.6 (FB)
- net FB_1V2: now reaches R15.2, R16.1, U4.6 (FB)
Other:
- moved on the sheet: R32
Changed lines of the file:
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@@
 	)
 	(junction
-		(at 223.52 105.41)
+		(at 100.33 106.68)
 		(diameter 0)
 		(color 0 0 0 0)
 	)
 	(junction
-		(at 100.33 106.68)
+		(at 212.09 53.34)
 		(diameter 0)
 		(color 0 0 0 0)
 	)
 	(junction
-		(at 212.09 53.34)
+		(at 223.52 105.41)
 		(diameter 0)
 		(color 0 0 0 0)
@@
 	(wire
 		(pts
-			(xy 218.44 105.41) (xy 223.52 105.41)
-		)
-		(stroke
-			(width 0)
-			(type default)
-		)
-	)
-	(wire
-		(pts
 			(xy 27.94 104.14) (xy 31.75 104.14)
 		)
@@
 	(wire
 		(pts
-			(xy 120.65 151.13) (xy 120.65 161.29)
+			(xy 223.52 105.41) (xy 228.6 105.41)
 		)
 		(stroke
@@
 	(wire
 		(pts
-			(xy 134.62 63.5) (xy 134.62 64.77)
+			(xy 120.65 151.13) (xy 120.65 161.29)
 		)
 		(stroke
@@
 	(wire
 		(pts
-			(xy 74.93 106.68) (xy 83.82 106.68)
+			(xy 134.62 63.5) (xy 134.62 64.77)
 		)
 		(stroke
@@
 	(wire
 		(pts
-			(xy 223.52 105.41) (xy 223.52 107.95)
+			(xy 74.93 106.68) (xy 83.82 106.68)
 		)
 		(stroke
@@
 	(wire
 		(pts
-			(xy 223.52 105.41) (xy 228.6 105.41)
+			(xy 223.52 111.76) (xy 223.52 113.03)
+		)
+		(stroke
+			(width 0)
+			(type default)
+		)
+	)
+	(wire
+		(pts
+			(xy 113.03 50.8) (xy 109.22 50.8)
 		)
 		(stroke
@@
 	(wire
 		(pts
-			(xy 109.22 57.15) (xy 109.22 50.8)
+			(xy 113.03 57.15) (xy 113.03 50.8)
 		)
 		(stroke
@@
 	(wire
 		(pts
+			(xy 218.44 105.41) (xy 223.52 105.41)
+		)
+		(stroke
+			(width 0)
+			(type default)
+		)
+	)
+	(wire
+		(pts
 			(xy 73.66 161.29) (xy 82.55 161.29)
 		)
@@
 	(wire
 		(pts
-			(xy 109.22 57.15) (xy 134.62 57.15)
+			(xy 113.03 57.15) (xy 134.62 57.15)
 		)
 		(stroke
@@
 	(wire
 		(pts
+			(xy 223.52 105.41) (xy 223.52 106.68)
+		)
+		(stroke
+			(width 0)
+			(type default)
+		)
+	)
+	(wire
+		(pts
 			(xy 129.54 45.72) (xy 129.54 48.26)
 		)
@@
 			"KShpbl9ib20geWVzKShvbl9ib2FyZCB5ZXMpKGRucCBubykodXVpZCAiMDlkMWM3OGUtN2QyMC00"
 			"YjRlLThiMGMtNTU4ZjgzMzc4ODViIikocHJvcGVydHkgICJSZWZlcmVuY2UiICJDMjIiIChhdCAx"
-			"NjUuMSAxMQ=="
+			"NjUuMSAxMQAAAAAAAAAAAAAAAAAAAAAAAAAAAAAAAAAAAAAAAAAAAAAAAAAAAAAAAAAAAAAAAAAA"
+			"AAAAAAAAAAAAAAAAAAAAAAAAAAAAAAAAAAAAAAAAAAAAAAAAAAAAAAAAAAAAAAAAAAAAAAAAAAAA"
+			"AAAAAAAAAAAAAAAAAAAAAAAAAAAAAAAAAAAAAAAAAAAAAAAAAAAAAAAAAAAAAAAAAAAAAAAAAAAA"
+			"AAAAAAAAAAAAAAAAAAAAAAAAAAAAAAAAAAAAAAAAAAAAAAAAAAAAAAAAAAAAAAAAAAAAAAAAAAAA"
+			"AAAAAAAAAAAAAAAAAAAAAAAAAAAAAAAAAAAAAAAAAAAAAAAAAAAAAAAAAAAAAAAAAAAAAAAAAAAA"
+			"AAAAAAAAAAAAAAAAAAAAAAAAAAAAAAAAAAAAAAAAAAAAAAAAAAAAAAAAAAAAAAAAAAAAAAAAAAAA"
+			"AAAAAAAAAAAAAAAAAAAAAAAAAAAAAAAAAAAAAAAAAAAAAAAAAAAAAAAAAAAAAAAAAAAAAAAAAAAA"
+			"AAAAAAAAAAAAAAAAAAAAAAAAAAAAAAAAAAAAAAAAAAAAAAAAAAAAAAAAAAAAAAAAAAAAAAAAAAAA"
+			"AAAAAAAAAAAAAAAAAAAAAAAAAAAAAAAAAAAAAAAAAAAAAAAAAAAAAAAAAAAAAAAAAAAAAAAAAAAA"
+			"AAAAAAAAAAAAAAAAAAAAAAAAAAAAAAAAAAAAAAAAAAAAAAAAAAAAAAAAAAAAAAAAAAAAAAAAAAAA"
+			"AAAAAAAAAAAAAAAAAAAAAAAAAAAAAAAAAAAAAAAAAAAAAAAAAAAAAAAAAAAAAAAAAAAAAAAAAAAA"
+			"AAAAAAAAAAAAAAAAAAAAAAAAAAAAAAAAAAAAAAAAAAAAAAAAAAAAAAAAAAAAAAAAAAAAAAAAAAAA"
+			"AAAAAAAAAAAAAAAAAAAAAAAAAAAAAAAAAAAAAAAAAAAAAAAAAAAAAAAAAAAAAAAAAAAAAAAAAAAA"
+			"AAAAAAAAAAAAAAAAAAAAAAAAAAAAAAAAAAAAAAAAAAAAAAAAAAAAAAAAAAAAAAAAAAAAAAAAAAAA"
+			"AAAAAAAAAAAAAAAAAAAAAAAAAAAAAAAAAAAAAAAAAAAAAAAAAAAAAAAAAAAAAAAAAAAAAAAAAAAA"
+			"AAAAAAAAAAAAAAAAAAAAAAAAAAAAAAAAAAAAAAAAAAAAAAAAAAAAAAAAAAAAAAAAAAAAAAAAAAAA"
+			"AAAAAAAAAAAAAAAAAAAAAAAAAAAAAAAAAAAAAAAAAAAAAAAAAAAAAAAAAAAAAAAAAAAAAAAAAAAA"
+			"AAAAAAAAAAAAAAAAAAAAAAAAAAAAAAAAAAAAAAAAAAAAAAAAAAAAAAAAAAAAAAAAAAAAAAAAAAAA"
+			"AAAAAAAAAA=="
 		)
 	)
@@
 	)
 	(label "FB_Vccint"
-		(at 111.76 57.15 0)
+		(at 276.86 57.15 0)
+		(effects
+			(font
+				(size 0.635 0.635)
+			)
+			(justify left bottom)
+		)
+	)
+	(label "FB_Vccint"
+		(at 119.38 57.15 0)
 		(effects
 			(font
@@
 		)
 	)
+	(label "FB_1V2"
+		(at 85.09 170.18 0)
+		(effects
+			(font
+				(size 0.635 0.635)
+			)
+			(justify left bottom)
+		)
+	)
 	(label "PG_Vccaux"
 		(at 46.99 170.18 0)
@@
 		)
 	)
+	(label "FB_3V3"
+		(at 208.28 119.38 0)
+		(effects
+			(font
+				(size 0.635 0.635)
+			)
+			(justify left bottom)
+		)
+	)
 	(label "EN_Vccint"
 		(at 33.02 45.72 180)
@@
 		)
 	)
+	(label "FB_1V35"
+		(at 85.09 120.65 0)
+		(effects
+			(font
+				(size 0.635 0.635)
+			)
+			(justify left bottom)
+		)
+	)
 	(label "PG_Vccaux"
 		(at 170.18 114.3 0)
@@
 		(polyline
 			(pts
-				(xy 194.31 24.13) (xy 194.31 77.724) (xy 328.041 78.486) (xy 328.295 24.638)
+				(xy 15.24 138.43) (xy 15.24 192.786) (xy 134.62 192.913) (xy 134.62 138.303)
 			)
 			(stroke
@@
 		(polyline
 			(pts
-				(xy 15.24 138.43) (xy 15.24 192.786) (xy 134.62 192.913) (xy 134.62 138.303)
+				(xy 138.43 83.82) (xy 138.3665 133.096) (xy 257.8735 133.604) (xy 257.81 83.82)
 			)
 			(stroke
@@
 		(polyline
 			(pts
-				(xy 138.43 83.82) (xy 138.3665 133.096) (xy 257.8735 133.604) (xy 257.81 83.82)
+				(xy 194.31 24.13) (xy 194.31 77.724) (xy 328.041 78.486) (xy 328.295 24.638)
 			)
 			(stroke
@@
 	(symbol
 		(lib_id "!Misc:R_15K_0603")
-		(at 223.52 110.49 0)
+		(at 223.52 109.22 0)
 		(unit 1)
 		(exclude_from_sim no)
@@
 		(fields_autoplaced yes)
 		(property "Reference" "R32"
-			(at 226.06 109.2199 0)
+			(at 226.06 107.9499 0)
 			(effects
 				(font
@@
 		)
 		(property "Value" "15K"
-			(at 226.06 111.7599 0)
+			(at 226.06 110.4899 0)
 			(effects
 				(font
@@
 		)
 		(property "Footprint" "Resistor_SMD:R_0603_1608Metric"
-			(at 223.52 110.49 0)
+			(at 223.52 109.22 0)
 			(effects
 				(font
@@
 		)
 		(property "Datasheet" "~"
-			(at 223.52 110.49 0)
+			(at 223.52 109.22 0)
 			(effects
 				(font
@@
 		)
 		(property "Description" "15K 0603 Resistor"
-			(at 223.52 110.49 0)
+			(at 223.52 109.22 0)
 			(effects
 				(font
@@
 		)
 		(property "LCSC Part #" "C22809"
-			(at 223.52 110.49 0)
+			(at 223.52 109.22 0)
 			(effects
 				(font
@@
 		)
 		(property "Digi-Key Part Number" "RES SMD 15K OHM 1% 1/10W 0603"
-			(at 223.52 110.49 0)
+			(at 223.52 109.22 0)
 			(effects
 				(font

Commit message: Add netnames for rails
Connections:
- net +Vccaux renamed +1V8
- net +Vccint renamed +1V0
Changed lines of the file:
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@@
 			"AAAAAAAAAAAAAAAAAAAAAAAAAAAAAAAAAAAAAAAAAAAAAAAAAAAAAAAAAAAAAAAAAAAAAAAAAAAA"
 			"AAAAAAAAAAAAAAAAAAAAAAAAAAAAAAAAAAAAAAAAAAAAAAAAAAAAAAAAAAAAAAAAAAAAAAAAAAAA"
+			"AAAAAAAAAAAAAAAAAAAAAAAAAAAAAAAAAAAAAAAAAAAAAAAAAAAAAAAAAAAAAAAAAAAAAAAAAAAA"
+			"AAAAAAAAAAAAAAAAAAAAAAAAAAAAAAAAAAAAAAAAAAAAAAAAAAAAAAAAAAAAAAAAAAAAAAAAAAAA"
+			"AAAAAAAAAAAAAAAAAAAAAAAAAAAAAAAAAAAAAAAAAAAAAAAAAAAAAAAAAAAAAAAAAAAAAAAAAAAA"
+			"AAAAAAAAAAAAAAAAAAAAAAAAAAAAAAAAAAAAAAAAAAAAAAAAAAAAAAAAAAAAAAAAAAAAAAAAAAAA"
+			"AAAAAAAAAAAAAAAAAAAAAAAAAAAAAAAAAAAAAAAAAAAAAAAAAAAAAAAAAAAAAAAAAAAAAAAAAAAA"
+			"AAAAAAAAAAAAAAAAAAAAAAAAAAAAAAAAAAAAAAAAAAAAAAAAAAAAAAAAAAAAAAAAAAAAAAAAAAAA"
+			"AAAAAAAAAAAAAAAAAAAAAAAAAAAAAAAAAAAAAAAAAAAAAAAAAAAAAAAAAAAAAAAAAAAAAAAAAAAA"
+			"AAAAAAAAAAAAAAAAAAAAAAAAAAAAAAAAAAAAAAAAAAAAAAAAAAAAAAAAAAAAAAAAAAAAAAAAAAAA"
+			"AAAAAAAAAAAAAAAAAAAAAAAAAAAAAAAAAAAAAAAAAAAAAAAAAAAAAAAAAAAAAAAAAAAAAAAAAAAA"
+			"AAAAAAAAAAAAAAAAAAAAAAAAAAAAAAAAAAAAAAAAAAAAAAAAAAAAAAAAAAAAAAAAAAAAAAAAAAAA"
+			"AAAAAAAAAAAAAAAAAAAAAAAAAAAAAAAAAAAAAAAAAAAAAAAAAAAAAAAAAAAAAAAAAAAAAAAAAAAA"
+			"AAAAAAAAAAAAAAAAAAAAAAAAAAAAAAAAAAAAAAAAAAAAAAAAAAAAAAAAAAAAAAAAAAAAAAAAAAAA"
+			"AAAAAAAAAAAAAAAAAAAAAAAAAAAAAAAAAAAAAAAAAAAAAAAAAAAAAAAAAAAAAAAAAAAAAAAAAAAA"
+			"AAAAAAAAAAAAAAAAAAAAAAAAAAAAAAAAAAAAAAAAAAAAAAAAAAAAAAAAAAAAAAAAAAAAAAAAAAAA"
+			"AAAAAAAAAAAAAAAAAAAAAAAAAAAAAAAAAAAAAAAAAAAAAAAAAAAAAAAAAAAAAAAAAAAAAAAAAAAA"
+			"AAAAAAAAAAAAAAAAAAAAAAAAAAAAAAAAAAAAAAAAAAAAAAAAAAAAAAAAAAAAAAAAAAAAAAAAAAAA"
+			"AAAAAAAAAAAAAAAAAAAAAAAAAAAAAAAAAAAAAAAAAAAAAAAAAAAAAAAAAAAAAAAAAAAAAAAAAAAA"
+			"AAAAAAAAAAAAAAAAAAAAAAAAAAAAAAAAAAAAAAAAAAAAAAAAAAAAAAAAAAAAAAAAAAAAAAAAAAAA"
 			"AAAAAAAAAA=="
 		)
@@
 		(polyline
 			(pts
-				(xy 138.43 83.82) (xy 138.3665 133.096) (xy 257.8735 133.604) (xy 257.81 83.82)
+				(xy 194.31 24.13) (xy 194.31 77.724) (xy 328.041 78.486) (xy 328.295 24.638)
 			)
 			(stroke
@@
 		(polyline
 			(pts
-				(xy 39.37 24.13) (xy 39.37 77.724) (xy 170.307 77.724) (xy 170.561 23.876)
+				(xy 138.43 83.82) (xy 138.3665 133.096) (xy 257.8735 133.604) (xy 257.81 83.82)
 			)
 			(stroke
@@
 		(polyline
 			(pts
-				(xy 15.24 83.82) (xy 15.1765 133.096) (xy 134.6835 133.604) (xy 134.62 83.82)
+				(xy 39.37 24.13) (xy 39.37 77.724) (xy 170.307 77.724) (xy 170.561 23.876)
 			)
 			(stroke
@@
 		(polyline
 			(pts
-				(xy 15.24 138.43) (xy 15.24 192.786) (xy 134.62 192.913) (xy 134.62 138.303)
+				(xy 15.24 83.82) (xy 15.1765 133.096) (xy 134.6835 133.604) (xy 134.62 83.82)
 			)
 			(stroke
@@
 		(polyline
 			(pts
-				(xy 194.31 24.13) (xy 194.31 77.724) (xy 328.041 78.486) (xy 328.295 24.638)
+				(xy 15.24 138.43) (xy 15.24 192.786) (xy 134.62 192.913) (xy 134.62 138.303)
 			)
 			(stroke
@@
 			)
 		)
-		(property "Component Class" "REG_Vccaux"
+		(property "Component Class" "REG_1V8"
 			(at 195.072 21.844 0)
 			(effects
@@
 			)
 		)
-		(property "Component Class" "REG_Vccint"
+		(property "Component Class" "REG_1V0"
 			(at 40.132 21.844 0)
 			(effects
@@
 	)
 	(symbol
-		(lib_id "power:GND")
-		(at 223.52 125.73 0)
+		(lib_id "power:+1V0")
+		(at 157.48 38.1 0)
 		(unit 1)
 		(exclude_from_sim no)
@@
 		(on_board yes)
 		(dnp no)
-		(fields_autoplaced yes)
-		(property "Reference" "#PWR053"
-			(at 223.52 132.08 0)
+		(property "Reference" "#PWR051"
+			(at 157.48 41.91 0)
 			(effects
 				(font
@@
 			)
 		)
-		(property "Value" "GND"
-			(at 223.52 130.81 0)
+		(property "Value" "+1V0"
+			(at 157.48 33.02 0)
 			(effects
 				(font
@@
 		)
 		(property "Footprint" ""
-			(at 223.52 125.73 0)
+			(at 157.48 38.1 0)
 			(effects
 				(font
@@
 		)
 		(property "Datasheet" ""
-			(at 223.52 125.73 0)
+			(at 157.48 38.1 0)
 			(effects
 				(font
@@
 			)
 		)
-		(property "Description" "Power symbol creates a global label with name \"GND\" , ground"
-			(at 223.52 125.73 0)
+		(property "Description" "Power symbol creates a global label with name \"+1V0\""
+			(at 157.48 38.1 0)
 			(effects
 				(font
@@
 			(project "aup"
 				(path "/312a869c-f247-4883-8e23-bdad51e1754f/018ff12c-0df9-4a4e-a203-c003842112a1"
-					(reference "#PWR053")
+					(reference "#PWR051")
 					(unit 1)
 				)
@@
 	)
 	(symbol
-		(lib_id "power:+5V")
-		(at 52.07 38.1 0)
+		(lib_id "power:GND")
+		(at 223.52 125.73 0)
 		(unit 1)
 		(exclude_from_sim no)
@@
 		(dnp no)
 		(fields_autoplaced yes)
-		(property "Reference" "#PWR017"
-			(at 52.07 41.91 0)
+		(property "Reference" "#PWR053"
+			(at 223.52 132.08 0)
 			(effects
 				(font
@@
 			)
 		)
-		(property "Value" "+5V"
-			(at 52.07 33.02 0)
+		(property "Value" "GND"
+			(at 223.52 130.81 0)
 			(effects
 				(font
@@
 		)
 		(property "Footprint" ""
-			(at 52.07 38.1 0)
+			(at 223.52 125.73 0)
 			(effects
 				(font
@@
 		)
 		(property "Datasheet" ""
-			(at 52.07 38.1 0)
+			(at 223.52 125.73 0)
 			(effects
 				(font
@@
 			)
 		)
-		(property "Description" "Power symbol creates a global label with name \"+5V\""
-			(at 52.07 38.1 0)
+		(property "Description" "Power symbol creates a global label with name \"GND\" , ground"
+			(at 223.52 125.73 0)
 			(effects
 				(font
@@
 			(project "aup"
 				(path "/312a869c-f247-4883-8e23-bdad51e1754f/018ff12c-0df9-4a4e-a203-c003842112a1"
-					(reference "#PWR017")
+					(reference "#PWR053")
 					(unit 1)
 				)
@@
 	)
 	(symbol
-		(lib_id "power:+1V0")
-		(at 157.48 38.1 0)
+		(lib_id "power:+5V")
+		(at 52.07 38.1 0)
 		(unit 1)
 		(exclude_from_sim no)
@@
 		(on_board yes)
 		(dnp no)
-		(property "Reference" "#PWR037"
-			(at 157.48 41.91 0)
+		(fields_autoplaced yes)
+		(property "Reference" "#PWR017"
+			(at 52.07 41.91 0)
 			(effects
 				(font
@@
 			)
 		)
-		(property "Value" "+Vccint"
-			(at 157.48 33.02 0)
+		(property "Value" "+5V"
+			(at 52.07 33.02 0)
 			(effects
 				(font
@@
 		)
 		(property "Footprint" ""
-			(at 157.48 38.1 0)
+			(at 52.07 38.1 0)
 			(effects
 				(font
@@
 		)
 		(property "Datasheet" ""
-			(at 157.48 38.1 0)
+			(at 52.07 38.1 0)
 			(effects
 				(font
@@
 			)
 		)
-		(property "Description" "Power symbol creates a global label with name \"+1V0\""
-			(at 157.48 38.1 0)
+		(property "Description" "Power symbol creates a global label with name \"+5V\""
+			(at 52.07 38.1 0)
 			(effects
 				(font
@@
 		)
 		(instances
-			(project ""
+			(project "aup"
 				(path "/312a869c-f247-4883-8e23-bdad51e1754f/018ff12c-0df9-4a4e-a203-c003842112a1"
-					(reference "#PWR037")
+					(reference "#PWR017")
 					(unit 1)
 				)
@@
 			)
 		)
-		(property "Value" "+Vccaux"
+		(property "Value" "+1V8"
 			(at 314.96 33.02 0)
 			(effects

Commit message: Start of regulator rework
Parts:
- removed C10: 0.1uf/50v, Capacitor_SMD:C_0603_1608Metric, symbol !Misc:C_0.1uf_0603
- removed C17: 0.1uf, Capacitor_SMD:C_0402_1005Metric, symbol !Misc:C_0.1uf_0402
- removed C18: 22uf/25V, Capacitor_SMD:C_0805_2012Metric, symbol !Misc:C_22uf_0805
- removed C8, C9: 10uf/50V, Capacitor_SMD:C_0805_2012Metric, symbol !Misc:C_10uf_0805
- removed L2: 1uH/2A, Inductor_SMD:L_1008_2520Metric, symbol !Misc:L_1uh_3A
- removed L7: 2.2uH/2A, Inductor_SMD:L_1008_2520Metric, symbol !Misc:L_2.2uh_3A
- removed R12: 10K, Resistor_SMD:R_0603_1608Metric, symbol !Misc:R_10K_0603
- removed R15, R16: 51K, Resistor_SMD:R_0603_1608Metric, symbol !Misc:R_51K_0603
- removed U4: TPS563257DRLR, !Misc:SOT6_DRL_TEX, symbol !Misc:TPS563257DRLR
- added C13, C15: 10uf/50V, Capacitor_SMD:C_0805_2012Metric, symbol !Misc:C_10uf_0805
- added L4: 2.2uH/5A, Inductor_SMD:L_Sunlord_MWSA0518S, symbol !Misc:L_2.2uh_5A
- added Q2: AO3400A, Package_TO_SOT_SMD:SOT-23, symbol !Misc:AO3400A
- added Q3: AO3401A, Package_TO_SOT_SMD:SOT-23, symbol !Misc:AO3401A
- added R11, R18: 2.2K, Resistor_SMD:R_0603_1608Metric, symbol !Misc:R_2.2K_0603
- added R21, R37: 10K, Resistor_SMD:R_0603_1608Metric, symbol !Misc:R_10K_0603
- added U6: ISL80103IRAJZ-TK, !Misc:DFN10_3X3_INR, symbol !Misc:ISL80103IRAJZ-TK
Connections:
- net +1V0: no longer R17.2
- net +1V2: now also C13.1, R11.1, U6.1 (VOUT), U6.2 (VOUT)
- net +1V35: no longer R24.2
- net +1V8: no longer R28.2
- net +3V3: now also C15.1, L4.2, Q3.2 (S), R21.1, R37.1, U6.10 (VIN), U6.9 (VIN)
- net +5V: now also R17.2, R24.2, R28.2
- net GND: now also C13.2, C15.2, Q2.2 (S), R18.2, U6.11 (EPAD), U6.5 (GND)
- net PG_Vccaux: now also Q2.1 (G)
- net SW_3V3: now also L4.1
- new net: Q2.3 (D), Q3.1 (G), R37.2
- new net: R11.2, R18.1, U6.3 (ADJ)
- new net: R21.2, U6.7 (ENABLE)
- new net +X3V3: Q3.3 (D)
- no-connect marks 0 -> 3
Other:
- note removed: "1v8 would ideally use a 1.5uh inductor, but weren't widely available in 1008. 2.2 is used for Vccaux to prioritize lowering ripple over transient response. Resistors use JLCPCB basic parts only. Used in series where exact matches could not be found, e.g. I couldn't find a FB pair with just 2 resistors, so did 25K and 20K, and used series resistors for the 25K."
- note removed: "Inductor selection: L = (Vout × (Vin - Vout)) / (Vin × ΔIL × f_sw) where ΔIL ≈ 0.3 × Iout Feedback resistor selection: Vout = 0.6 × (1 + Rt / Rb) → Rt / Rb = Vout / 0.6 - 1 → Rt = Rb × (Vout / 0.6 - 1) Enable resistor selection: EN max V is 5.5 max. If feeding from a voltage source, use a voltage divider to stay under this max. Venh (enable is true) max: 1.25V Venl (enable is false) min: 0.9V If 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"
- note removed: "Layout notes from datasheet: https://www.ti.com/lit/ds/symlink/tps563252.pdf • Keep VIN and GND traces as wide as possible to reduce trace impedance. • Place the input capacitor and output capacitor as close to the device as possible to minimize trace impedance. • Provide sufficient vias for the input capacitor and output capacitor. • Keep the SW trace as physically short and wide as practical to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"
