File: pcb/aup/ddr3.kicad_sch (KiCad schematic)
At the start: 1 part, among them IC1 MT41K128M16JT-125_K

Commit message: Very rough assigment for DDR to banks
Parts:
- added R16, R21: 1K, Resistor_SMD:R_0603_1608Metric, symbol !Misc:R_1K_0603
Connections:
- net +1V35: now reaches IC1.A1 (VDDQ_1)
- net +1V35: now also IC1.A8 (VDDQ_2), IC1.B2 (VDD_1), IC1.C1 (VDDQ_3), IC1.C9 (VDDQ_4), IC1.D2 (VDDQ_5), IC1.D9 (VDD_2), IC1.E9 (VDDQ_6), IC1.F1 (VDDQ_7), IC1.G7 (VDD_3), IC1.H2 (VDDQ_8), IC1.H9 (VDDQ_9), IC1.K2 (VDD_4), IC1.K8 (VDD_5), IC1.N1 (VDD_6), IC1.N9 (VDD_7), IC1.R1 (VDD_8), IC1.R9 (VDD_9), R16.1
- net DDR_DQ13: now reaches IC1.A2 (DQ13)
- net DDR_DQ15: now reaches IC1.A3 (DQ15)
- net DDR_DQ12: now reaches IC1.A7 (DQ12)
- net GND: now reaches IC1.A9 (VSS_1)
- net GND: now also IC1.B1 (VSSQ_1), IC1.B3 (VSS_2), IC1.B9 (VSSQ_2), IC1.D1 (VSSQ_3), IC1.D8 (VSSQ_4), IC1.E1 (VSS_3), IC1.E2 (VSSQ_5), IC1.E8 (VSSQ_6), IC1.F9 (VSSQ_7), IC1.G1 (VSSQ_8), IC1.G8 (VSS_4), IC1.G9 (VSSQ_9), IC1.J2 (VSS_5), IC1.J8 (VSS_6), IC1.M1 (VSS_7), IC1.M9 (VSS_8), IC1.P1 (VSS_9), IC1.P9 (VSS_10), IC1.T1 (VSS_11), IC1.T9 (VSS_12), R21.2
- net DDR_UQDS_N: now reaches IC1.B7 (UDQS#)
- net DDR_DQ14: now reaches IC1.B8 (DQ14)
- net DDR_DQ11: now reaches IC1.C2 (DQ11)
- net DDR_DQ9: now reaches IC1.C3 (DQ9)
- net DDR_UDQS_P: now reaches IC1.C7 (UDQS)
- net DDR_DQ10: now reaches IC1.C8 (DQ10)
- net DDR_DM1: now reaches IC1.D3 (UDM)
- net DDR_DQ8: now reaches IC1.D7 (DQ8)
- net DDR_DQ0: now reaches IC1.E3 (DQ0)
- net DDR_DM0: now reaches IC1.E7 (LDM)
- net DDR_DQ2: now reaches IC1.F2 (DQ2)
- net DDR_LDQS_P: now reaches IC1.F3 (LDQS)
- net DDR_DQ1: now reaches IC1.F7 (DQ1)
- net DDR_DQ3: now reaches IC1.F8 (DQ3)
- net DDR_DQ6: now reaches IC1.G2 (DQ6)
- net DDR_LDQS_N: now reaches IC1.G3 (LDQS#)
- net +V075: now reaches IC1.H1 (VREFDQ)
- net +V075: now also IC1.M8 (VREFCA), R16.2, R21.1
- net DDR_DQ4: now reaches IC1.H3 (DQ4)
- net DDR_DQ7: now reaches IC1.H7 (DQ7)
- net DDR_DQ5: now reaches IC1.H8 (DQ5)
- net DDR_RAS: now reaches IC1.J3 (RAS#)
- net DDR_CK_P: now reaches IC1.J7 (CK)
- net DDR_ODT: now reaches IC1.K1 (ODT)
- net DDR_CAS: now reaches IC1.K3 (CAS#)
- net DDR_CK_N: now reaches IC1.K7 (CK#)
- net DDR_CKE: now reaches IC1.K9 (CKE)
- net DDR_CS: now reaches IC1.L2 (CS#)
- net DDR_WE: now reaches IC1.L3 (WE#)
- net DDR_A10: now reaches IC1.L7 (A10/AP)
- net DDR_BA0: now reaches IC1.M2 (BA0)
- net DDR_BA2: now reaches IC1.M3 (BA2)
- net DDR_A3: now reaches IC1.N2 (A3)
- net DDR_A0: now reaches IC1.N3 (A0)
- net DDR_A12: now reaches IC1.N7 (A12/BC#)
- net DDR_BA1: now reaches IC1.N8 (BA1)
- net DDR_A5: now reaches IC1.P2 (A5)
- net DDR_A2: now reaches IC1.P3 (A2)
- net DDR_A1: now reaches IC1.P7 (A1)
- net DDR_A4: now reaches IC1.P8 (A4)
- net DDR_A7: now reaches IC1.R2 (A7)
- net DDR_A9: now reaches IC1.R3 (A9)
- net DDR_A11: now reaches IC1.R7 (A11)
- net DDR_A6: now reaches IC1.R8 (A6)
- net DDR_RST: now reaches IC1.T2 (RESET#)
- net DDR_A13: now reaches IC1.T3 (A13)
- net DDR_A8: now reaches IC1.T8 (A8)
- no-connect marks 0 -> 6
Other:
- note added: "add 220+240R"
- note added: "need rst pulldown, caps, res between ck_n and ck_p, termination?"
- moved on the sheet: IC1
