File: pcb/aup/ddr3.kicad_sch (KiCad schematic)
At the start: 3 parts, among them IC1 MT41K128M16JT-125_K

Commit message: Add hierarchical sheets for banks and add caps.
There are some stale sheets in this commit, but I don't want to delete
an active one accidentally. Save them all for now, and then go back and
clean them up.
Other:
- note added: "???"
Changed lines of the file:
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@@
+		)
+	)
+	(text "???\n"
+		(exclude_from_sim no)
+		(at 240.792 27.686 0)
+		(effects
+			(font
+				(size 5.08 5.08)
+				(thickness 1.016)
+				(bold yes)
+				(color 255 0 0 1)
+			)
 		)
 	)
