File: pcb/aup/ext_power.kicad_sch (KiCad schematic)
At the start: 29 parts, among them J5 Conn_01x02_Pin, Q1 AO3401A, U10 TPS2116DRLR, U2 USBLC6-2SC6, U3 TPS563257DRLR

Commit message: Switch to 50 pin sockets
Parts:
- renumbered J5 to J13
Changed lines of the file:
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@@
 		(dnp no)
 		(fields_autoplaced yes)
-		(property "Reference" "J5"
+		(property "Reference" "J13"
 			(at 254 43.1799 0)
 			(effects
@@
 			(project "aup"
 				(path "/312a869c-f247-4883-8e23-bdad51e1754f/66f6f111-4301-4b77-9bf5-52f6219d7e81"
-					(reference "J5")
+					(reference "J13")
 					(unit 1)
 				)

Commit message: More upsized planning
Parts:
- removed BJ1: Barral_Jack_12V, Connector_BarrelJack:BarrelJack_Horizontal, symbol !Misc:Barral_Jack_12V
- removed C2, C3: 10uf/50V, Capacitor_SMD:C_0805_2012Metric, symbol !Misc:C_10uf_0805
- removed C4: 0.1uf/50v, Capacitor_SMD:C_0603_1608Metric, symbol !Misc:C_0.1uf_0603
- removed C5: 33pf, Capacitor_SMD:C_0402_1005Metric, symbol !Misc:C_33pf_0402
- removed C6, C8: 0.1uf, Capacitor_SMD:C_0402_1005Metric, symbol !Misc:C_0.1uf_0402
- removed C7: 22uf/25V, Capacitor_SMD:C_0805_2012Metric, symbol !Misc:C_22uf_0805
- removed F1: 2A, Fuse:Fuse_1812_4532Metric, symbol !Misc:Fuse_16V_2A_1812
- removed L1: 2.2uH/5A, Inductor_SMD:L_Sunlord_MWSA0518S, symbol !Misc:L_2.2uh_5A
- removed Q1: AO3401A, Package_TO_SOT_SMD:SOT-23, symbol !Misc:AO3401A
- removed R10, R6: 20K, Resistor_SMD:R_0603_1608Metric, symbol !Misc:R_20K_0603
- removed R4, R7, R9: 10K, Resistor_SMD:R_0603_1608Metric, symbol !Misc:R_10K_0603
- removed R5: 100K, Resistor_SMD:R_0603_1608Metric, symbol !Misc:R_100K_0603
- removed R8: 150K, Resistor_SMD:R_0603_1608Metric, symbol !Misc:R_150K_0603
- removed U3: TPS563257DRLR, !Misc:SOT6_DRL_TEX, symbol !Misc:TPS563257DRLR
Connections:
- net +5V: no longer J13.2 (Pin_2)
- net REG_5V renamed Ext5V
- net Ext5V: now also J13.2 (Pin_2)
- no-connect marks 4 -> 3
Other:
- moved on the sheet: J13
